File: display.sch (KiCad schematic (older format))
At the start: 27 parts, among them J6 AVR-ISP-6, Q2 MMBT3904, Q3 MMBT3904, Q4 MMBT3904, Q5 MMBT3904, U5 SC56-11GWA, U6 SC56-11GWA, U7 ATmega48P-20MMHR, U8 SC56-11GWA, U9 SC56-11GWA

Commit message: Main Board Rev A files
Parts:
- added C4, C8: 16pF, Capacitor_SMD:C_0603_1608Metric, symbol Device:C
- added Y1: Crystal_GND24, Crystal:Crystal_SMD_3225-4Pin_3.2x2.5mm, symbol Device:Crystal_GND24
Connections:
- wire segments 105 -> 115
- no-connect marks 4 -> 6
Other:
- moved on the sheet: C2, R21, R22, R23, R24, R25, R26, R27, R28
